File: Hardware/JTAG_HW_FT2232HL/JTAG_HW.kicad_sch (KiCad schematic)
At the start: 36 parts, among them J1 Conn_01x10_Pin, J6 USB_C16PIN, U1 93CxxC, U3 NUP2202, U4 FT2232HL, U5 XC6206PxxxMR, Y2 Crystal_GND24

Commit message: Remove elements
Parts:
- removed FB1, FB2: FerriteBead_Small, Inductor_SMD:L_0805_2012Metric_Pad1.15x1.40mm_HandSolder, symbol Device:FerriteBead_Small
- removed R6, R7: 27, Resistor_SMD:R_0805_2012Metric_Pad1.20x1.40mm_HandSolder, symbol Device:R_Small
- removed U3: NUP2202, Package_TO_SOT_SMD:SOT-363_SC-70-6, symbol Power_Protection:NUP2202
- added R6, R7: R, symbol Device:R
Connections:
- net +5V: now also R6.1, R7.1
- net 3.3V: now also U4.4 (VPHY), U4.9 (VPLL)
- net at J6.A5 (CC1): now also R7.2
- net D-: now reaches J6.A6 (D+), J6.B6 (D+)
- net D-: now also U4.8 (DP)
- net D+: now reaches J6.A7 (D-), J6.B7 (D-)
- net D+: now also U4.7 (DM)
- net at J6.B5 (CC2): now also R6.2
- no-connect marks 25 -> 23
Other:
- note removed: "27Ом резисторы - лишнии"
- note removed: "Подтянуть CC к 5V через резистор 5.1кОм (именно этот номинал)"
- note removed: "Посадочное место перепроверить"
- note removed: "Убрать индуктивность. FT советуют, но тогда еще нужны развязывающие кондеры, уже много и сложно"
